File: Armed.kicad_pcb (KiCad board)
At the start: 2 copper layers, 100 x 71 mm, 344 parts, among them J10 GS3, J11 Conn_01x04, J12 GS3, J14 Conn_01x03, J15 Conn_01x03, J16 GS3, J17 GS3, J18 GS3, J19 GS3, J20 USB_B, J21 GS3, J22 GS3, J23 GS3, J24 GS3, J25 GS3, J26 GS3, J27 GS3, J28 GS3, J29 GS3, J30 GS3, J31 GS3, J6 Conn_01x03, J7 Conn_01x04, J8 GS3, J9 Conn_01x06, SW1 SW_SPST, U1 STM32F407V(E-G)Tx, U2 24LC512, U3 74HCT02, U5 AMS1117-3.3, Y1 8MHz

Commit message: Armed 1.1
Parts:
- removed the C34 at (131.1, 52.4)
- removed the C36 at (146.7, 93.3)
- removed the C37 at (146.7, 95.3)
- removed the C38 at (146.7, 97.3)
- removed the C39 at (146.7, 99.2)
- removed the D5 at (93.6, 71.0)
- removed D9: RND SS110F-AT, complib:DO-219AB
- removed J10, J12, J16, J17, J18, J19, J21, J22, J23, J24, J25, J26, J27, J28, J29, J30, J31, J8: GS3, Connectors:GS3
- removed the R33 at (149.9, 43.7)
- removed the R6 at (99.5, 66.4)
- removed the R8 at (98.3, 69.4)
- removed REF** (x180): VIA-0.6mm, VIA-0.6mm
- removed the TR3 at (159.2, 98.8)
- removed the U5 at (141.2, 50.3)
- added C1: 10nF, Capacitors_SMD:C_0805, F.Cu at (94.4, 48.2)
- added C14: 100nF, Capacitors_SMD:C_0805, F.Cu at (108.3, 68.7)
- added C2: 10nF, Capacitors_SMD:C_0805, F.Cu at (103.4, 48.2)
- added C4: 1uF 16V X7R/X5R, Capacitors_SMD:C_0805, F.Cu at (138.2, 57.5)
- added C50: 1uF, Capacitors_SMD:C_0805, F.Cu at (129.2, 52.4)
- added C53: 100nF, Capacitors_SMD:C_0805, F.Cu at (122.9, 52.4)
- added C54: 20pF, Capacitors_SMD:C_0805, F.Cu at (135.9, 68.5)
- added C55: 20pF, Capacitors_SMD:C_0805, F.Cu at (135.9, 64.4)
- added C56: 100nF, Capacitors_SMD:C_0805, F.Cu at (142.8, 53.7)
- added D10: 1N4148WS, Diodes_SMD:D_SOD-323, F.Cu at (165.3, 102.4)
- added D11: 1N4148WS, Diodes_SMD:D_SOD-323, F.Cu at (160.3, 102.4)
- added D6: 1N4148WS, Diodes_SMD:D_SOD-323, F.Cu at (170.9, 102.4)
- added I2C1: Conn_01x04, Pin_Headers:Pin_Header_Straight_2x02_Pitch2.54mm, F.Cu at (94.7, 79.5)
- added JP1: USB-VCC, Jumper:SolderJumper-2_P1.3mm_Open_RoundedPad1.0x1.5mm, B.Cu at (94.7, 70.7)
- added JP10: E0-MISO, Jumper:SolderJumper-2_P1.3mm_Open_RoundedPad1.0x1.5mm, B.Cu at (137.7, 83.7)
- added JP11: E0-MOSI, Jumper:SolderJumper-2_P1.3mm_Open_RoundedPad1.0x1.5mm, B.Cu at (130.2, 83.7)
- added JP12: E0-SCK, Jumper:SolderJumper-2_P1.3mm_Open_RoundedPad1.0x1.5mm, B.Cu at (132.7, 83.7)
- added JP13: E0-CS, Jumper:SolderJumper-2_P1.3mm_Open_RoundedPad1.0x1.5mm, B.Cu at (135.2, 83.7)
- added JP14: X-MISO, Jumper:SolderJumper-2_P1.3mm_Open_RoundedPad1.0x1.5mm, B.Cu at (92.0, 83.7)
- added JP15: X-MOSI, Jumper:SolderJumper-2_P1.3mm_Open_RoundedPad1.0x1.5mm, B.Cu at (84.5, 83.7)
- added JP16: X-SCK, Jumper:SolderJumper-2_P1.3mm_Open_RoundedPad1.0x1.5mm, B.Cu at (87.0, 83.7)
- added JP17: X-CS, Jumper:SolderJumper-2_P1.3mm_Open_RoundedPad1.0x1.5mm, B.Cu at (89.5, 83.7)
- added JP18: Y-MISO, Jumper:SolderJumper-2_P1.3mm_Open_RoundedPad1.0x1.5mm, B.Cu at (107.2, 83.7)
- added JP19: Y-MOSI, Jumper:SolderJumper-2_P1.3mm_Open_RoundedPad1.0x1.5mm, B.Cu at (99.7, 83.7)
- added JP2: E1-MISO, Jumper:SolderJumper-2_P1.3mm_Open_RoundedPad1.0x1.5mm, B.Cu at (152.9, 83.7)
- added JP20: Y-SCK, Jumper:SolderJumper-2_P1.3mm_Open_RoundedPad1.0x1.5mm, B.Cu at (102.2, 83.7)
- added JP21: Y-CS, Jumper:SolderJumper-2_P1.3mm_Open_RoundedPad1.0x1.5mm, B.Cu at (104.7, 83.7)
- added JP22: Z-MISO, Jumper:SolderJumper-2_P1.3mm_Open_RoundedPad1.0x1.5mm, B.Cu at (122.5, 83.8)
- added JP23: Z-MOSI, Jumper:SolderJumper-2_P1.3mm_Open_RoundedPad1.0x1.5mm, B.Cu at (115.0, 83.8)
- added JP24: Z-SCK, Jumper:SolderJumper-2_P1.3mm_Open_RoundedPad1.0x1.5mm, B.Cu at (117.5, 83.8)
- added JP25: Z-CS, Jumper:SolderJumper-2_P1.3mm_Open_RoundedPad1.0x1.5mm, B.Cu at (120.0, 83.8)
- added JP26: E0-CFG0, Jumper:SolderJumper-3_P1.3mm_Open_RoundedPad1.0x1.5mm, B.Cu at (136.8, 90.8)
- added JP27: X-CFG0, Jumper:SolderJumper-3_P1.3mm_Open_RoundedPad1.0x1.5mm, B.Cu at (91.0, 90.8)
- added JP28: Y-CFG0, Jumper:SolderJumper-3_P1.3mm_Open_RoundedPad1.0x1.5mm, B.Cu at (106.3, 90.8)
- added JP29: Z-CFG0, Jumper:SolderJumper-3_P1.3mm_Open_RoundedPad1.0x1.5mm, B.Cu at (121.5, 90.8)
- added JP3: E1-MOSI, Jumper:SolderJumper-2_P1.3mm_Open_RoundedPad1.0x1.5mm, B.Cu at (145.4, 83.7)
- added JP30: E0-MS1, Jumper:SolderJumper-3_P1.3mm_Open_RoundedPad1.0x1.5mm, B.Cu at (136.8, 98.9)
- added JP31: X-MS1, Jumper:SolderJumper-3_P1.3mm_Open_RoundedPad1.0x1.5mm, B.Cu at (91.0, 98.9)
- added JP32: Y-MS1, Jumper:SolderJumper-3_P1.3mm_Open_RoundedPad1.0x1.5mm, B.Cu at (106.3, 98.9)
- added JP33: Z-MS1, Jumper:SolderJumper-3_P1.3mm_Open_RoundedPad1.0x1.5mm, B.Cu at (121.5, 98.9)
- added JP34: X-MS2, Jumper:SolderJumper-3_P1.3mm_Open_RoundedPad1.0x1.5mm, B.Cu at (91.0, 96.1)
- added JP35: Y-MS2, Jumper:SolderJumper-3_P1.3mm_Open_RoundedPad1.0x1.5mm, B.Cu at (106.3, 96.2)
- added JP36: Z-MS2, Jumper:SolderJumper-3_P1.3mm_Open_RoundedPad1.0x1.5mm, B.Cu at (121.5, 96.2)
- added JP37: E0-MS2, Jumper:SolderJumper-3_P1.3mm_Open_RoundedPad1.0x1.5mm, B.Cu at (136.8, 96.2)
- added JP38: X-MS3, Jumper:SolderJumper-3_P1.3mm_Open_RoundedPad1.0x1.5mm, B.Cu at (91.0, 93.5)
- added JP39: Y-MS3, Jumper:SolderJumper-3_P1.3mm_Open_RoundedPad1.0x1.5mm, B.Cu at (106.3, 93.5)
- added JP4: E1-SCK, Jumper:SolderJumper-2_P1.3mm_Open_RoundedPad1.0x1.5mm, B.Cu at (147.9, 83.7)
- added JP40: Z-MS3, Jumper:SolderJumper-3_P1.3mm_Open_RoundedPad1.0x1.5mm, B.Cu at (121.5, 93.5)
- added JP41: E0-MS3, Jumper:SolderJumper-3_P1.3mm_Open_RoundedPad1.0x1.5mm, B.Cu at (136.8, 93.5)
- added JP42: I2C-VCC, Jumper:SolderJumper-3_P1.3mm_Open_RoundedPad1.0x1.5mm, B.Cu at (107.3, 67.7)
- added JP5: E1-CS, Jumper:SolderJumper-2_P1.3mm_Open_RoundedPad1.0x1.5mm, B.Cu at (150.4, 83.7)
- added JP6: E1-CFG0, Jumper:SolderJumper-3_P1.3mm_Open_RoundedPad1.0x1.5mm, B.Cu at (152.0, 90.8)
- added JP7: E1-MS1, Jumper:SolderJumper-3_P1.3mm_Open_RoundedPad1.0x1.5mm, B.Cu at (152.0, 98.9)
- added JP8: E1-MS2, Jumper:SolderJumper-3_P1.3mm_Open_RoundedPad1.0x1.5mm, B.Cu at (152.0, 96.2)
- added JP9: E1-MS3, Jumper:SolderJumper-3_P1.3mm_Open_RoundedPad1.0x1.5mm, B.Cu at (152.0, 93.5)
- added L2: 7427920415, Inductors_SMD:L_0805, F.Cu at (120.3, 52.4)
- added R13: 47k, Resistors_SMD:R_0805, F.Cu at (145.3, 62.7)
- added R26: 9.53k, Resistors_SMD:R_0805, F.Cu at (136.1, 50.5)
- added R29: 10k, Resistors_SMD:R_0805, F.Cu at (151.9, 99.2)
- added R31: 4k7, Resistors_SMD:R_0805, F.Cu at (108.3, 72.4)
- added R34: 4k7, Resistors_SMD:R_0805, F.Cu at (136.7, 97.3)
- added R36: 4k7, Resistors_SMD:R_0805, F.Cu at (106.2, 97.3)
- added R37: 4k7, Resistors_SMD:R_0805, F.Cu at (121.5, 97.3)
- added R38: 10k, Resistors_SMD:R_0805, F.Cu at (90.9, 99.3)
- added R39: 10k, Resistors_SMD:R_0805, F.Cu at (106.2, 99.2)
- added R40: 10k, Resistors_SMD:R_0805, F.Cu at (121.5, 99.2)
- added R41: 10k, Resistors_SMD:R_0805, F.Cu at (136.7, 99.2)
- added R42: 20, Resistors_SMD:R_0805, F.Cu at (99.8, 68.7)
- added R45: 4k7, Resistors_SMD:R_0805, F.Cu at (97.6, 68.7)
- added R46: 100k, Resistors_SMD:R_0805, F.Cu at (104.1, 72.4)
- added R48: 47k, Resistors_SMD:R_0805, F.Cu at (147.8, 43.6)
- added R49: 47k, Resistors_SMD:R_0805, F.Cu at (149.8, 43.6)
- added SER1: Conn_02x02, Pin_Headers:Pin_Header_Straight_2x02_Pitch2.54mm, F.Cu at (101.1, 79.5)
- added TR6: PMV40UN2, TO_SOT_Packages_SMD:SOT-23, F.Cu at (159.2, 98.8)
- added U3: AOZ1282CI/AP3012, Package_TO_SOT_SMD:SOT-23-6, F.Cu at (139.0, 49.6)
- added U4: 24LC32AT-I/OT, Package_TO_SOT_SMD:SOT-23-5, F.Cu at (105.1, 68.7)
- C10, C11: value 10uF -> 2.2uF; footprint Capacitors_Tantalum_SMD:CP_Tantalum_Case-A_EIA-3216-18_Reflow -> Capacitors_SMD:C_0805
- C12: value 2.2uF -> 100nF; footprint Resistors_SMD:R_0805 -> Capacitors_SMD:C_0805
- C13: value 2.2uF -> 10uF 16V (X5R/X7R); footprint Resistors_SMD:R_0805 -> Capacitors_SMD:C_0805
- C15, C16, C17: value 2.2uF -> 1nF; footprint Resistors_SMD:R_0805 -> Capacitors_SMD:C_0805
- C18, C21, C23, C24, C25, C26, C27, C28, C35: value 100nF -> 1nF; footprint Resistors_SMD:R_0805 -> Capacitors_SMD:C_0805
- C19: value 20pF -> 100uF 35V; footprint Resistors_SMD:R_0805 -> Capacitors_SMD:CP_Elec_6.3x5.8
- C20: value 10pF -> 1nF; footprint Resistors_SMD:R_0805 -> Capacitors_SMD:C_0805
- C22, C29, C30, C31: footprint Resistors_SMD:R_0805 -> Capacitors_SMD:C_0805
- C3: value 100uF -> 10nF; footprint Capacitors_SMD:CP_Elec_6.3x5.8 -> Capacitors_SMD:C_0805
- C32, C33: value 1uF -> 1nF; footprint Resistors_SMD:R_0805 -> Capacitors_SMD:C_0805
- C34: renamed from C50; footprint Resistors_SMD:R_0805 -> Capacitors_SMD:C_0805
- C36: renamed from C2; value 100uF -> 100uF 35V
- C37: renamed from C4; value 100uF -> 100uF 35V
- C38: renamed from C5; value 100uF -> 100uF 35V
- C39: renamed from C1; value 100uF -> 100uF 35V
- C40, C42: value 1nF -> 2.2uF; footprint Resistors_SMD:R_0805 -> Capacitors_SMD:C_0805
- C41, C43, C44, C45, C46, C47, C48: value 1nF -> 100nF; footprint Resistors_SMD:R_0805 -> Capacitors_SMD:C_0805
- C49: value 1nF -> 10uF; footprint Resistors_SMD:R_0805 -> Capacitors_SMD:C_0805
- C5: renamed from C14; value 100uF -> 100uF 35V
- C51: value 1nF -> 1uF; footprint Resistors_SMD:R_0805 -> Capacitors_SMD:C_0805
- C52: value 10uF -> 100nF; footprint Resistors_SMD:R_0805 -> Capacitors_SMD:C_0805
- C6: value 100nF -> 1uF 16V X7R/X5R; footprint Resistors_SMD:R_0805 -> Capacitors_SMD:C_0805
- C7: value 10nF -> 100nF; footprint Resistors_SMD:R_0805 -> Capacitors_SMD:C_0805
- C8: value 10nF -> 10uF 35V (X5R/X7R); footprint Resistors_SMD:R_0805 -> Capacitors_SMD:C_0805
- C9: value 10nF -> 2.2uF; footprint Resistors_SMD:R_0805 -> Capacitors_SMD:C_0805
- D1: value RND SS110F-AT -> BAT60J; footprint complib:DO-219AB -> Diodes_SMD:D_SMA
- D8: value RND SS110F-AT -> B140-13-F; footprint complib:DO-219AB -> Diodes_SMD:D_SMA
- F1: renamed from F2; value Fuse -> 3557-2
- F2: renamed from F1; value Fuse -> 3557-2
- L1: value 7427920415 -> 22uH NR6028T220M; footprint Resistors_SMD:R_0805 -> Inductors_SMD:L_Taiyo-Yuden_NR-60xx
- R10: renamed from R18; value 4K7 -> 4k7
- R12: renamed from R14; value 4K7 -> 4k7
- R14: renamed from R34; value 4K7 -> 4k7
- R18: renamed from R20; value 10k -> 4k7
- R21: renamed from R23; value 4k7 -> 10k
- R25: value R -> 49.9k
- R27: value 100k -> 4k7
- R30: renamed from R24; value R -> 4k7
- R35: renamed from R5; value 100k -> 4k7
- R9: renamed from R13; value 4K7 -> 4k7
- SWD1: value CONN_02X04 -> Conn_02X04
- U2: value 24LC512 -> AP2112K-3.3TRG1; footprint Housings_SOIC:SOIC-8_3.9x4.9mm_Pitch1.27mm -> Package_TO_SOT_SMD:SOT-23-5
- moved D1 82.6 mm to (94.7, 70.5), turned to 270 degrees
- moved C21 64.9 mm to (100.9, 93.3), turned to 0 degrees
- moved C32 64.0 mm to (85.7, 99.3), turned to 0 degrees
- moved C28 62.2 mm to (85.7, 97.3), turned to 0 degrees
- moved C24 59.6 mm to (85.7, 95.3), turned to 0 degrees
- moved C20 58.0 mm to (85.7, 93.3), turned to 0 degrees
- moved D8 57.8 mm to (142.8, 49.1), turned to 270 degrees
- moved C49 55.2 mm to (135.2, 55.9)
- moved C15 53.8 mm to (146.7, 93.3), turned to 0 degrees
- moved C7 53.5 mm to (145.3, 64.7)
- moved C33 52.5 mm to (100.9, 99.2), turned to 0 degrees
- moved C16 52.3 mm to (146.7, 95.3), turned to 0 degrees
- moved C19 51.7 mm to (87.6, 86.9)
- moved C17 51.6 mm to (146.7, 97.3), turned to 0 degrees
- moved R27 51.1 mm to (151.9, 97.3), turned to 180 degrees
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- renumbered A5 to A1, A1 to A2, A2 to A3, A3 to A4, A4 to A5, D4 to D3, D3 to D4, D7 to D5, D6 to D7, FAN11 to FAN2, FAN21 to FAN3, J9 to J1, J7 to J2, J6 to J3, J14 to J4, J15 to J5, J20 to J6, J11 to J7, R9 to R1, R12 to R11, R29 to R15, R15 to R16, R19 to R17, R21 to R19, R16 to R2, R22 to R20, R35 to R22, R32 to R23, R30 to R24, R31 to R28, R36 to R3, R1 to R32, R2 to R33, R37 to R4, R7 to R43, R26 to R44, R28 to R47, R38 to R5, R10 to R6, R11 to R7, R17 to R8, TEMP0 to TEMP1, TEMP1 to TEMP2, TEMP2 to TEMP3, TR4 to TR1, TR5 to TR2, TR6 to TR3, TR1 to TR4, TR2 to TR5, U3 to U1, U1 to U5, Z-MOT2 to Z-MOT1, Z-MOT1 to Z-MOT2
Connections:
- A1 pad 10: DRV_MOSI -> Net-(A1-Pad10)
- A1 pad 11: DRV_SCK -> Net-(A1-Pad11)
- A1 pad 12: E1_CS_PIN -> Net-(A1-Pad12)
- A1 pad 13: DRV_MISO -> Net-(A1-Pad13)
- A1 pad 3: Net-(A5-Pad3) -> Net-(A1-Pad3)
- A1 pad 4: Net-(A5-Pad4) -> Net-(A1-Pad4)
- A1 pad 5: Net-(A5-Pad5) -> Net-(A1-Pad5)
- A1 pad 6: Net-(A5-Pad6) -> Net-(A1-Pad6)
- A2 pad 10: DRV_MOSI -> Net-(A2-Pad10)
- A2 pad 11: DRV_SCK -> Net-(A2-Pad11)
- A2 pad 12: X_CS_PIN -> Net-(A2-Pad12)
- A2 pad 13: DRV_MISO -> Net-(A2-Pad13)
- A2 pad 3: Net-(A1-Pad3) -> Net-(A2-Pad3)
- A2 pad 4: Net-(A1-Pad4) -> Net-(A2-Pad4)
- A2 pad 5: Net-(A1-Pad5) -> Net-(A2-Pad5)
- A2 pad 6: Net-(A1-Pad6) -> Net-(A2-Pad6)
- A3 pad 10: DRV_MOSI -> Net-(A3-Pad10)
- A3 pad 11: DRV_SCK -> Net-(A3-Pad11)
- A3 pad 12: Y_CS_PIN -> Net-(A3-Pad12)
- A3 pad 13: DRV_MISO -> Net-(A3-Pad13)
- A3 pad 3: Net-(A2-Pad3) -> Net-(A3-Pad3)
- A3 pad 4: Net-(A2-Pad4) -> Net-(A3-Pad4)
- A3 pad 5: Net-(A2-Pad5) -> Net-(A3-Pad5)
- A3 pad 6: Net-(A2-Pad6) -> Net-(A3-Pad6)
- A4 pad 10: DRV_MOSI -> Net-(A4-Pad10)
- A4 pad 11: DRV_SCK -> Net-(A4-Pad11)
- A4 pad 12: Z_CS_PIN -> Net-(A4-Pad12)
- A4 pad 13: DRV_MISO -> Net-(A4-Pad13)
- A4 pad 3: Net-(A3-Pad3) -> Net-(A4-Pad3)
- A4 pad 4: Net-(A3-Pad4) -> Net-(A4-Pad4)
- A4 pad 5: Net-(A3-Pad5) -> Net-(A4-Pad5)
- A5 pad 10: DRV_MOSI -> Net-(A5-Pad10)
- A5 pad 11: DRV_SCK -> Net-(A5-Pad11)
- A5 pad 12: E0_CS_PIN -> Net-(A5-Pad12)
- A5 pad 13: DRV_MISO -> Net-(A5-Pad13)
- A5 pad 3: Net-(A4-Pad3) -> Net-(A5-Pad3)
- A5 pad 4: Net-(A4-Pad4) -> Net-(A5-Pad4)
- A5 pad 5: Net-(A4-Pad5) -> Net-(A5-Pad5)
- A5 pad 6: Net-(A4-Pad6) (its old number) -> Net-(A5-Pad6)
- C10 pad 1: +5V -> TEMP_1_PIN
- C11 pad 1: +3V3 -> TEMP_2_PIN
- C12 pad 1: GND -> Net-(C12-Pad1)
- C12 pad 2: VCAP_1 -> Net-(C12-Pad2)
- C13 pad 1: GND -> +5V
- C13 pad 2: VCAP_2 -> GND
- C15 pad 1: TEMP_0_PIN -> Net-(A1-Pad3)
- C16 pad 1: TEMP_1_PIN -> Net-(A1-Pad4)
- C17 pad 1: TEMP_2_PIN -> Net-(A1-Pad5)
- C18 pad 1: RESET -> Net-(A1-Pad6)
- C19 pad 1: GND -> 12V1
- C19 pad 2: Net-(C19-Pad2) -> GND
- C20 pad 1: GND -> Net-(A2-Pad3)
- C20 pad 2: Net-(C20-Pad2) -> GND
- C21 pad 1: POWER_MONITOR -> Net-(A3-Pad3)
- C22 pad 1: Net-(A1-Pad3) -> Net-(A4-Pad3)
- C23 pad 1: GND -> Net-(A5-Pad3)
- C23 pad 2: +3V3 -> GND
- C24 pad 1: GND -> Net-(A2-Pad4)
- C24 pad 2: +3V3 -> GND
- C25 pad 1: GND -> Net-(A3-Pad4)
- C25 pad 2: +3V3 -> GND
- C26 pad 1: GND -> Net-(A4-Pad4)
- C26 pad 2: +3V3 -> GND
- C27 pad 1: GND -> Net-(A5-Pad4)
- C27 pad 2: +3V3 -> GND
- C28 pad 1: GND -> Net-(A2-Pad5)
- C28 pad 2: +3V3 -> GND
- C29 pad 1: Net-(A1-Pad4) -> Net-(A3-Pad5)
- C3 pad 1: 12V1 -> Z_MIN_PIN
- C30 pad 1: Net-(A1-Pad5) -> Net-(A4-Pad5)
- C31 pad 1: Net-(A1-Pad6) -> Net-(A5-Pad5)
- C32 pad 1: GND -> Net-(A2-Pad6)
- C32 pad 2: VREF+ -> GND
- C33 pad 1: VDDA -> Net-(A3-Pad6)
- C35 pad 1: VDDA -> Net-(A5-Pad6)
- C40 pad 1: Net-(A2-Pad3) -> GND
- C40 pad 2: GND -> VCAP_1
- C41 pad 1: Net-(A3-Pad3) -> RESET
- C42 pad 1: Net-(A4-Pad3) -> GND
- C42 pad 2: GND -> VCAP_2
- C43 pad 1: Net-(A2-Pad4) -> GND
- C43 pad 2: GND -> +3V3
- C44 pad 1: Net-(A3-Pad4) -> GND
- C44 pad 2: GND -> +3V3
- C45 pad 1: Net-(A4-Pad4) -> GND
- C45 pad 2: GND -> +3V3
- C46 pad 1: Net-(A2-Pad5) -> GND
- C46 pad 2: GND -> +3V3
- C47 pad 1: Net-(A3-Pad5) -> GND
- C47 pad 2: GND -> +3V3
- C48 pad 1: Net-(A4-Pad5) -> GND
- C48 pad 2: GND -> +3V3
- C49 pad 1: Net-(A2-Pad6) -> GND
- C49 pad 2: GND -> +3V3
- C51 pad 1: Net-(A4-Pad6) (its old number) -> VDDA
- C52 pad 2: +3V3 -> VREF+
- C7 pad 1: X_MIN_PIN -> POWER_MONITOR
- C8 pad 1: Y_MIN_PIN -> 12V1
- C9 pad 1: Z_MIN_PIN -> TEMP_0_PIN
- D1 pad 1: 12V1 -> +5V
- D1 pad 2: FAN0- -> Net-(D1-Pad2)
- D8 pad 1: 12V1 -> Net-(C12-Pad2)
- D8 pad 2: FAN1- -> GND
- E0-MOT1 pad 1: Net-(A4-Pad3) -> Net-(A5-Pad3)
- E0-MOT1 pad 2: Net-(A4-Pad4) -> Net-(A5-Pad4)
- E0-MOT1 pad 3: Net-(A4-Pad5) -> Net-(A5-Pad5)
- E0-MOT1 pad 4: Net-(A4-Pad6) (its old number) -> Net-(A5-Pad6)
- E1-MOT1 pad 1: Net-(A5-Pad3) -> Net-(A1-Pad3)
- E1-MOT1 pad 2: Net-(A5-Pad4) -> Net-(A1-Pad4)
- E1-MOT1 pad 3: Net-(A5-Pad5) -> Net-(A1-Pad5)
- E1-MOT1 pad 4: Net-(A5-Pad6) -> Net-(A1-Pad6)
- J3 pad 3: +3V3 -> +5V
- J4 pad 3: +3V3 -> +5V
- J5 pad 3: +3V3 -> +5V
- J6 pad 1: Net-(D5-Pad2) (its old number) -> Net-(D1-Pad2)
- L1 pad 1: VDDA -> +5V
- L1 pad 2: +3V3 -> Net-(C12-Pad2)
- R25 pad 1: SCL -> +5V
- R25 pad 2: +3V3 -> Net-(R25-Pad2)
- R27 pad 1: GND -> Net-(JP6-Pad1)
- R27 pad 2: BOOT0 -> +3V3
- R30 pad 2: +3V3 -> /VCC_I2C
- R35 pad 1: DRV_MISO -> Net-(JP27-Pad1)
- SW1 pad 1: GND -> RESET
- SW1 pad 2: RESET -> GND
- SWD1 pad 3: RX_PIN -> Net-(SWD1-Pad3)
- SWD1 pad 4: TX_PIN -> SWO
- U2 pad 1: GND -> +5V
- U2 pad 3: GND -> +5V
- U2 pad 4: GND -> Net-(U2-Pad4)
- U2 pad 5: SDA -> +3V3
- U5 pad 12: Net-(C19-Pad2) -> Net-(C54-Pad2)
- U5 pad 13: Net-(C20-Pad2) -> Net-(C55-Pad2)
- U5 pad 46: (no net) -> Net-(U5-Pad46)
- U5 pad 5: (no net) -> Net-(U5-Pad5)
- U5 pad 6: (no net) -> Net-(U5-Pad6)
- U5 pad 60: (no net) -> Net-(U5-Pad60)
- U5 pad 61: (no net) -> Net-(U5-Pad61)
- U5 pad 62: (no net) -> Net-(U5-Pad62)
- U5 pad 68: (no net) -> Net-(U5-Pad68)
- U5 pad 7: (no net) -> Net-(U5-Pad7)
- U5 pad 8: (no net) -> Net-(U5-Pad8)
- U5 pad 80: (no net) -> E0_ENABLE_PIN
- U5 pad 89: E0_ENABLE_PIN -> SWO
- U5 pad 9: (no net) -> Net-(U5-Pad9)
- X-MOT1 pad 1: Net-(A1-Pad3) -> Net-(A2-Pad3)
- X-MOT1 pad 2: Net-(A1-Pad4) -> Net-(A2-Pad4)
- X-MOT1 pad 3: Net-(A1-Pad5) -> Net-(A2-Pad5)
- X-MOT1 pad 4: Net-(A1-Pad6) -> Net-(A2-Pad6)
- Y-MOT1 pad 1: Net-(A2-Pad3) -> Net-(A3-Pad3)
- Y-MOT1 pad 2: Net-(A2-Pad4) -> Net-(A3-Pad4)
- Y-MOT1 pad 3: Net-(A2-Pad5) -> Net-(A3-Pad5)
- Y-MOT1 pad 4: Net-(A2-Pad6) -> Net-(A3-Pad6)
- Y1 pad 1: Net-(C19-Pad2) -> Net-(C54-Pad2)
- Y1 pad 2: Net-(C20-Pad2) -> Net-(C55-Pad2)
- Z-MOT1 pad 1: Net-(A3-Pad3) -> Net-(A4-Pad3)
- Z-MOT1 pad 2: Net-(A3-Pad4) -> Net-(A4-Pad4)
- Z-MOT1 pad 3: Net-(A3-Pad5) -> Net-(A4-Pad5)
- Z-MOT2 pad 1: Net-(A3-Pad3) -> Net-(A4-Pad3)
- Z-MOT2 pad 2: Net-(A3-Pad4) -> Net-(A4-Pad4)
- Z-MOT2 pad 3: Net-(A3-Pad5) -> Net-(A4-Pad5)
Routing:
- net DRV_MOSI: track 179.7 -> 0.00 mm, vias 4 -> 0
- net DRV_SCK: track 146.7 -> 0.00 mm, vias 10 -> 0
- net DRV_MISO: track 118.0 -> 0.00 mm, vias 5 -> 0
- net GND: track 753.5 -> 665.5 mm, vias 20 -> 227
- net SPI_MOSI: track 90.0 -> 171.6 mm, vias 4 -> 11
- net SPI_MISO: track 81.4 -> 146.1 mm, vias 4 -> 13
- net SPI_SCK: track 82.8 -> 143.4 mm, vias 4 -> 6
- net +5V: track 160.4 -> 202.4 mm, vias 3 -> 5
- net /VCC_I2C: track 0.00 -> 26.4 mm, vias 0 -> 1
- net Net-(A1-Pad10): track 0.00 -> 22.9 mm, vias 0 -> 2
- net Net-(A4-Pad10): track 0.00 -> 22.7 mm, vias 0 -> 4
- net Net-(A5-Pad10): track 0.00 -> 22.3 mm, vias 0 -> 2
- net Net-(A3-Pad10): track 0.00 -> 22.1 mm, vias 0 -> 2
- net Net-(D7-Pad2): track 1.84 -> 23.9 mm, vias 0 -> 2
- net Net-(A2-Pad10): track 0.00 -> 21.3 mm, vias 0 -> 2
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Other:
- net class 3V3: clearance 0.2 -> 0.1524; via_dia 0.7372 -> 0.6
- net class 5V: clearance 0.2 -> 0.1524; via_dia 0.7372 -> 0.6
- net class Default: via_dia 0.4572 -> 0.508; via_drill 0.1524 -> 0.2
- net class GND: clearance 0.2 -> 0.1524; via_dia 0.7372 -> 0.6
- net class HIGH_CURRENT: clearance 0.2 -> 0.1524
- net class MEDIUM_CURRENT: clearance 0.2 -> 0.1524
- net class MOTOR: clearance 0.2 -> 0.1524
- rule via_min_drill: 0.1524 -> 0.2
- rule via_min_size: 0.4572 -> 0.508
- board text added: "+"
- board text added: "+ FAN0 -"
- board text added: "+ FAN1 -"
- board text added: "+ FAN2 -"
- board text added: "-"
- board text added: "- BED +"
- board text added: "- HEATER0 +"
- board text added: "- HEATER1 +"
- board text added: "2018-10-02 Rev 1.1"
- board text added: "3V3"
- board text added: "5V"
- board text added: "BOOT0"
- board text added: "ENDSTOPS"
- board text added: "EXT0"
- board text added: "EXT1"
- board text added: "EXT2"
- board text added: "EXT3"
- board text added: "EXT4"
- board text added: "EXT5"
- board text added: "EXT6"
- board text added: "EXT7"
- board text added: "EXT8"
- board text added: "EXT9"
- board text added: "FAN0 ↑"
- board text added: "FS"
- board text added: "GND"
- board text added: "HEATERS"
- board text added: "I2C-VCC"
- board text added: "MISO"
- board text added: "MOSI"
- board text added: "POWER SUPPLY (MAX 24V)"
- board text added: "PSON"
- board text added: "RX"
- board text added: "SCK"
- board text added: "SCL"
- board text added: "SDA"
- board text added: "SWCLK"
- board text added: "SWDIO"
- board text added: "SWO"
- board text added: "T0"
- board text added: "T1"
- board text added: "TBED"
- board text added: "TEMPERATURE SENSORS"
- board text added: "TX"
- board text added: "USB-VCC"
- board text added: "VCC-I2C"
- board text added: "VIN"
- board text added: "X"
- board text added: "Y"
- board text added: "Z"
- board text added: "↑ T0"
- board text added: "↑ TBED"
- board text removed: "2018-02-15 Rev 1.0"
- board text removed: "FAN3 ↑"
- board text removed: "MS1"
- board text removed: "MS2"
- board text removed: "MS3"
- board text removed: "↑ T2"
- board text removed: "↑ T3"
